File: AudioInterface/AudioInterface.kicad_pcb (KiCad board)
At the start: 2 copper layers, 88.1 x 68.3 mm, 29 parts, among them J1 Capsule, J2 Set_Gain, J3 Audio_Out, J4 Power, J5 Conn_02x01_Row_Letter_First, J6 Conn_02x01_Row_Letter_First, U1 THAT1512, U2 NMA0515SC

Commit message: image
Routing:
- net /Bandpass-/B_OUT: track 63.2 -> 83.3 mm

Commit message: new start
Parts:
- removed J2: Set_Gain, Connector_JST:JST_EH_B2B-EH-A_1x02_P2.50mm_Vertical
- removed J3: Audio_Out, Connector_JST:JST_EH_B2B-EH-A_1x02_P2.50mm_Vertical
- removed J4: Power, Connector_JST:JST_EH_B2B-EH-A_1x02_P2.50mm_Vertical
- added H1: MountingHole_Pad, MountingHole:MountingHole_2.2mm_M2_DIN965_Pad_TopBottom, F.Cu at (106.7, 115.4)
- added H2: MountingHole_Pad, MountingHole:MountingHole_2.2mm_M2_DIN965_Pad_TopBottom, F.Cu at (187.8, 115.4)
- added H3: MountingHole_Pad, MountingHole:MountingHole_2.2mm_M2_DIN965_Pad_TopBottom, F.Cu at (106.7, 54.1)
- added H4: MountingHole_Pad, MountingHole:MountingHole_2.2mm_M2_DIN965_Pad_TopBottom, F.Cu at (187.8, 54.1)
- added R11: 5, Resistor_THT:R_Axial_DIN0207_L6.3mm_D2.5mm_P10.16mm_Horizontal, F.Cu at (108.6, 141.2)
- J1: value Capsule -> AudioAmp; footprint Connector_JST:JST_EH_B3B-EH-A_1x03_P2.50mm_Vertical -> Connector_FFC-FPC:Molex_200528-0090_1x09-1MP_P1.00mm_Horizontal
- moved R1 123.2 mm to (100.8, 147.1), turned to 0 degrees
- moved R3 109.6 mm to (100.8, 151.2), turned to 0 degrees
- moved C5 109.3 mm to (75.3, 159.4), turned to 0 degrees
- moved U1 106.4 mm to (101.3, 155.3), turned to 0 degrees
- moved R2 100.4 mm to (108.6, 137.1), turned to 0 degrees
- moved R5 98.9 mm to (86.4, 161.2), turned to 0 degrees
- moved C2 97.9 mm to (115.2, 147.1)
- moved C4 92.8 mm to (83.1, 138.1), turned to 0 degrees
- moved C1 90.4 mm to (123.0, 139.0), turned to 0 degrees
- moved R6 82.3 mm to (108.6, 133.1), turned to 0 degrees
- moved R4 78.5 mm to (121.9, 133.1), turned to 0 degrees
- moved C3 68.8 mm to (123.0, 146.8), turned to 0 degrees
- moved C9 56.9 mm to (117.8, 58.1)
- moved C10 50.7 mm to (112.6, 110.8), turned to 90 degrees
- moved C11 41.1 mm to (166.2, 58.3), turned to -90 degrees
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Connections:
- C1 pad 1: Net-(C1-Pad1) -> mic -
- C11 pad 1: GND -> INT_GND
- C2 pad 2: Net-(C2-Pad2) -> mic +
- C3 pad 1: Net-(C3-Pad1) -> Audio_out
- C4 pad 2: GND -> INT_GND
- C5 pad 1: GND -> INT_GND
- C6 pad 1: Net-(C6-Pad1) -> VBUS
- C6 pad 2: Net-(C6-Pad2) -> GND
- C7 pad 1: Net-(C6-Pad1) -> VBUS
- C7 pad 2: Net-(C6-Pad2) -> GND
- C9 pad 1: GND -> INT_GND
- J1 pad 1: Net-(C1-Pad1) -> GND
- J1 pad 2: GND -> mic +
- J1 pad 3: Net-(C2-Pad2) -> GND
- R1 pad 2: Net-(C1-Pad1) -> mic -
- R2 pad 1: Net-(C2-Pad2) -> mic +
- R3 pad 1: GND -> INT_GND
- R4 pad 2: GND -> INT_GND
- R5 pad 2: GND -> INT_GND
- R6 pad 1: GND -> INT_GND
- R7 pad 2: GND -> INT_GND
- R9 pad 2: GND -> INT_GND
- U1 pad 5: GND -> INT_GND
- U2 pad 1: Net-(C6-Pad1) -> VBUS
- U2 pad 2: Net-(C6-Pad2) -> GND
- U2 pad 5: GND -> INT_GND
Routing:
- net /Bandpass+/B_OUT: track 121.1 -> 0.00 mm
- net /Bandpass-/B_IN: track 97.7 -> 0.00 mm
- net /Bandpass-/B_OUT: track 83.3 -> 0.00 mm
- net VBUS: track 0.00 -> 43.9 mm
- net /Bandpass+/B_IN: track 43.7 -> 0.00 mm
- net Net-(C6-Pad2): track 41.4 -> 0.00 mm
- net Net-(C6-Pad1): track 40.6 -> 0.00 mm
- net Net-(C2-Pad1): track 29.3 -> 0.00 mm
- net GND: track 0.00 -> 27.2 mm, vias 12 -> 0
- net Net-(C1-Pad2): track 19.9 -> 0.00 mm
- net Net-(C8-Pad2): track 16.9 -> 0.00 mm
- net Net-(C10-Pad2): track 16.7 -> 0.00 mm
- net Net-(C1-Pad1): track 14.0 -> 0.00 mm
- net Net-(R11-Pad2): track 13.0 -> 0.00 mm
- net Net-(C3-Pad1): track 11.9 -> 0.00 mm
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- removed copper zone on B.Cu, net GND
- removed copper zone on F.Cu, net GND
