File: AudioInterface/AudioInterface.kicad_sch (KiCad schematic)
At the start: 19 parts, among them J1 Capsule, J2 Set_Gain, J3 Audio_Out, J4 Power, U1 THAT1512, U2 NMA0515SC

Commit message: new start
Parts:
- removed C1, C2: 22u, Capacitor_THT:C_Radial_D6.3mm_H11.0mm_P2.50mm, symbol Device:C_Small
- removed J1: Capsule, Connector_JST:JST_EH_B3B-EH-A_1x03_P2.50mm_Vertical, symbol Connector_Generic:Conn_01x03
- removed J2: Set_Gain, Connector_JST:JST_EH_B2B-EH-A_1x02_P2.50mm_Vertical, symbol Connector_Generic:Conn_01x02
- removed J3: Audio_Out, Connector_JST:JST_EH_B2B-EH-A_1x02_P2.50mm_Vertical, symbol Connector_Generic:Conn_01x02
- removed J4: Power, Connector_JST:JST_EH_B2B-EH-A_1x02_P2.50mm_Vertical, symbol Connector_Generic:Conn_01x02
- added H1, H2, H3, H4: MountingHole_Pad, MountingHole:MountingHole_2.2mm_M2_DIN965_Pad_TopBottom, symbol Mechanical:MountingHole_Pad
- added J1: AudioAmp, Connector_FFC-FPC:Molex_200528-0090_1x09-1MP_P1.00mm_Horizontal, symbol Connector:Conn_01x09_Male
- added R11: 5, Resistor_THT:R_Axial_DIN0207_L6.3mm_D2.5mm_P10.16mm_Horizontal, symbol Device:R
- C4, C5, C6, C7: footprint (none) -> Capacitor_THT:CP_Radial_D12.5mm_P5.00mm
- R1, R2, R5, R6: footprint (none) -> Resistor_THT:R_Axial_DIN0207_L6.3mm_D2.5mm_P10.16mm_Horizontal
- R3: value 3.9k -> (none)
- R4: value 3.9k -> 100; footprint (none) -> Resistor_THT:R_Axial_DIN0207_L6.3mm_D2.5mm_P10.16mm_Horizontal
- U2: footprint (none) -> Converter_DCDC:Converter_DCDC_Murata_NMAxxxxSC_THT
Connections:
- net Bandpass+/B_IN: now also C5.2, R2.2, R4.1, R6.2, U1.4 (V-); no longer U2.6 (VOUT+)
- net Bandpass+/B_OUT: now also U1.3 (+IN); no longer C4.1, R1.1, R5.1, U1.7 (V+)
- net Bandpass-/B_IN: now also C4.1, R1.1, R3.1, R5.1, U1.7 (V+); no longer U2.4 (VOUT-)
- net Bandpass-/B_OUT: now also U1.2 (-IN); no longer C5.2, R2.2, R6.2, U1.4 (V-)
- net GND: now also C6.2, C7.2, U2.2 (VIN-), J1.1 (Pin_1), J1.3 (Pin_3), J1.5 (Pin_5), J1.7 (Pin_7), J1.9 (Pin_9); no longer C4.2, C5.1, R3.1, R4.2, R5.2, R6.1, U1.5 (Ref), U2.5 (0V)
- net mic -: now reaches R1.2
- net mic -: now also J1.4 (Pin_4)
- net at R3.2: now also U2.6 (VOUT+); no longer U1.2 (-IN)
- net mic +: now reaches R2.1
- net mic +: now also J1.2 (Pin_2)
- net at U1.1 (Rg1): now also R11.2
- net at U1.8 (Rg2): now also R11.1
- net Audio_out: now reaches C3.1
- net Audio_out: now also J1.6 (Pin_6)
- net VBUS: now reaches C6.1, C7.1, U2.1 (VIN+)
- net VBUS: now also J1.8 (Pin_8)
- new net: R4.2, U2.4 (VOUT-)
- new net INT_GND: C4.2, C5.1, R5.2, R6.1, U1.5 (Ref), U2.5 (0V)
- new net Shield: H1.1, H2.1, H3.1, H4.1
Other:
- moved on the sheet: C3, C4, C5, C6, C7, R1, R2, R5, R6, U1, U2
