File: AudioInterface/Bandpass.kicad_sch (KiCad schematic)
At the start: 5 parts

Commit message: new start
Parts:
- C8: value (none) -> 270nF; footprint (none) -> Capacitor_THT:C_Rect_L18.0mm_W8.0mm_P15.00mm_FKS3_FKP3
- C9: footprint (none) -> Capacitor_THT:C_Rect_L18.0mm_W8.0mm_P15.00mm_FKS3_FKP3
- J5: value (none) -> Conn_02x01_Row_Letter_First; footprint (none) -> Connector_PinHeader_2.54mm:PinHeader_2x01_P2.54mm_Vertical
- R7: value (none) -> 20k; footprint (none) -> Resistor_THT:R_Axial_DIN0207_L6.3mm_D2.5mm_P10.16mm_Horizontal
- R8: footprint (none) -> Resistor_THT:R_Axial_DIN0207_L6.3mm_D2.5mm_P10.16mm_Horizontal
Connections:
- net GND renamed INT_GND
Changed lines of the file:
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@@
     (stroke (width 0) (type default) (color 0 0 0 0))
   )
-  (global_label "GND" (shape input) (at 91.44 67.31 270) (fields_autoplaced)
+  (global_label "INT_GND" (shape input) (at 91.44 67.31 270) (fields_autoplaced)
     (effects (font (size 1.27 1.27)) (justify right))
-    (property "Intersheet References" "${INTERSHEET_REFS}" (id 0) (at 91.3606 73.5047 90)
+    (property "Intersheet References" "${INTERSHEET_REFS}" (id 0) (at 91.3606 77.3752 90)
       (effects (font (size 1.27 1.27)) (justify right) hide)
     )
   )
-  (global_label "GND" (shape input) (at 120.65 67.31 270) (fields_autoplaced)
+  (global_label "INT_GND" (shape input) (at 120.65 67.31 270) (fields_autoplaced)
     (effects (font (size 1.27 1.27)) (justify right))
-    (property "Intersheet References" "${INTERSHEET_REFS}" (id 0) (at 120.5706 73.5047 90)
+    (property "Intersheet References" "${INTERSHEET_REFS}" (id 0) (at 120.5706 77.3752 90)
       (effects (font (size 1.27 1.27)) (justify right) hide)
     )
@@
     (in_bom yes) (on_board yes) (fields_autoplaced)
     (property "Reference" "J5" (id 0) (at 102.87 33.02 0))
-    (property "Value" "" (id 1) (at 102.87 35.56 0))
-    (property "Footprint" "" (id 2) (at 101.6 39.37 0)
+    (property "Value" "Conn_02x01_Row_Letter_First" (id 1) (at 102.87 35.56 0))
+    (property "Footprint" "Connector_PinHeader_2.54mm:PinHeader_2x01_P2.54mm_Vertical" (id 2) (at 101.6 39.37 0)
       (effects (font (size 1.27 1.27)) hide)
     )
@@
       (effects (font (size 1.27 1.27)) (justify left))
     )
-    (property "Value" "" (id 1) (at 93.218 64.643 0)
+    (property "Value" "20k" (id 1) (at 93.218 64.643 0)
       (effects (font (size 1.27 1.27)) (justify left))
     )
-    (property "Footprint" "" (id 2) (at 89.662 63.5 90)
+    (property "Footprint" "Resistor_THT:R_Axial_DIN0207_L6.3mm_D2.5mm_P10.16mm_Horizontal" (id 2) (at 89.662 63.5 90)
       (effects (font (size 1.27 1.27)) hide)
     )
@@
       (effects (font (size 1.27 1.27)) (justify left))
     )
-    (property "Footprint" "" (id 2) (at 120.65 64.77 0)
+    (property "Footprint" "Capacitor_THT:C_Rect_L18.0mm_W8.0mm_P15.00mm_FKS3_FKP3" (id 2) (at 120.65 64.77 0)
       (effects (font (size 1.27 1.27)) hide)
     )
@@
       (effects (font (size 1.27 1.27)) (justify left))
     )
-    (property "Footprint" "" (id 2) (at 113.03 56.388 90)
+    (property "Footprint" "Resistor_THT:R_Axial_DIN0207_L6.3mm_D2.5mm_P10.16mm_Horizontal" (id 2) (at 113.03 56.388 90)
       (effects (font (size 1.27 1.27)) hide)
     )
@@
       (effects (font (size 1.27 1.27)) (justify left))
     )
-    (property "Value" "" (id 1) (at 87.503 52.2732 0)
+    (property "Value" "270nF" (id 1) (at 87.503 52.2732 0)
       (effects (font (size 1.27 1.27)) (justify left))
     )
-    (property "Footprint" "" (id 2) (at 86.36 54.61 0)
+    (property "Footprint" "Capacitor_THT:C_Rect_L18.0mm_W8.0mm_P15.00mm_FKS3_FKP3" (id 2) (at 86.36 54.61 0)
       (effects (font (size 1.27 1.27)) hide)
     )
